File: top.sch (KiCad schematic (older format))
At the start: 27 parts, among them J1 USB_B_Mini, J2 TC2030_NL, J3 FFC-0.5MM-6POS, J4 Conn_01x02, J5 Conn_01x02, U1 PMIC-LDO-XC6204B332MR_SOT23-5_, U2 LP2985-5.0, U3 ATmega328P-MU, U4 ADXL335, Y1 16MHz

Commit message: Move BNC connectors to correct hemispheres
Positions within the hemisphere don’t matter.
Parts:
- J4: value Conn_01x02 -> Port_1
- J5: value Conn_01x02 -> Port_2
Changed lines of the file:
@@
 AR Path="/5C920754/5C99C62E" Ref="J5"  Part="1"
 F 0 "J5" H 5080 1242 50  0000 L CNN
-F 1 "Conn_01x02" H 5080 1151 50  0000 L CNN
+F 1 "Port_2" H 5080 1151 50  0000 L CNN
 F 2 "Connector_PinHeader_1.27mm:PinHeader_1x02_P1.27mm_Vertical" H 5000 1250 50  0001 C CNN
 F 3 "~" H 5000 1250 50  0001 C CNN
@@
 AR Path="/5C920754/5C99C634" Ref="J4"  Part="1"
 F 0 "J4" H 5080 792 50  0000 L CNN
-F 1 "Conn_01x02" H 5080 701 50  0000 L CNN
+F 1 "Port_1" H 5080 701 50  0000 L CNN
 F 2 "Connector_PinHeader_1.27mm:PinHeader_1x02_P1.27mm_Vertical" H 5000 800 50  0001 C CNN
 F 3 "~" H 5000 800 50  0001 C CNN

Commit message: Added initial tracks
Parts:
- U4: symbol SparkfunSensors:ADXL335 -> top-hemi-rescue:ADXL335-SparkfunSensors
Connections:
- net +5V_EXT: now also J2.6 (Pin_6); no longer J2.1 (Pin_1)
- net DTR: now also J1.2 (D-); no longer J1.3 (D+)
- net GND: now also J2.1 (Pin_1); no longer J1.6 (Shield), J2.6 (Pin_6)
- net MISO: now also J2.4 (Pin_4); no longer J2.3 (Pin_3)
- net MOSI: now also J2.5 (Pin_5); no longer J2.2 (Pin_2)
- net RXI: now also J1.3 (D+); no longer J1.2 (D-)
- net SCK: now also J2.3 (Pin_3); no longer J2.4 (Pin_4)
- net ~RST: now also J2.2 (Pin_2); no longer J2.5 (Pin_5)
Changed lines of the file:
@@
 $EndComp
 $Comp
-L SparkfunSensors:ADXL335 U?
+L top-hemi-rescue:ADXL335-SparkfunSensors U?
 U 1 1 5C9710AE
 P 8150 3150
@@
 L power:GND #PWR?
 U 1 1 5C9734D3
-P 2050 3900
+P 1550 3400
 AR Path="/5C9734D3" Ref="#PWR?"  Part="1"
 AR Path="/5C920754/5C9734D3" Ref="#PWR04"  Part="1"
-F 0 "#PWR04" H 2050 3650 50  0001 C CNN
-F 1 "GND" H 2055 3727 50  0000 C CNN
-F 2 "" H 2050 3900 50  0001 C CNN
-F 3 "" H 2050 3900 50  0001 C CNN
-	1    2050 3900
+F 0 "#PWR04" H 1550 3150 50  0001 C CNN
+F 1 "GND" H 1555 3227 50  0000 C CNN
+F 2 "" H 1550 3400 50  0001 C CNN
+F 3 "" H 1550 3400 50  0001 C CNN
+	1    1550 3400
 	1    0    0    -1
 $EndComp
@@
 Wire Wire Line
 	4800 1250 4500 1250
+Text Label 2050 3800 2    50   ~ 0
+MOSI
+Text Label 2050 3700 2    50   ~ 0
+MISO
+Text Label 2050 3600 2    50   ~ 0
+SCK
 Text Label 2050 3500 2    50   ~ 0
-MOSI
-Text Label 2050 3600 2    50   ~ 0
-MISO
-Text Label 2050 3700 2    50   ~ 0
-SCK
-Text Label 2050 3800 2    50   ~ 0
 ~RST
 Text Label 5550 2700 0    50   ~ 0
@@
 Text Label 6300 3900 0    50   ~ 0
 DTR
+Text Label 2150 5050 0    50   ~ 0
+DTR
 Text Label 2150 4950 0    50   ~ 0
-DTR
-Text Label 2150 5050 0    50   ~ 0
 RXI
 Text Label 2150 5150 0    50   ~ 0
@@
 Wire Wire Line
 	950  2550 1050 2550
-Text Label 2050 3400 2    50   ~ 0
+Text Label 2050 3900 2    50   ~ 0
 +5V_EXT
 Text HLabel 4000 6650 0    50   Input ~ 0
@@
 	1    0    0    -1
 $EndComp
-Wire Wire Line
-	1750 5350 1850 5350
-Connection ~ 1850 5350
 $Comp
 L MCU_Microchip_ATmega:ATmega328P-MU U3
@@
 	1    0    0    -1
 $EndComp
+Wire Wire Line
+	1550 3400 2050 3400
 $EndSCHEMATC

Commit message: Changed to 2.54mm
Parts:
- D2, D3: footprint Connector_PinHeader_1.27mm:PinHeader_1x04_P1.27mm_Vertical -> Connector_PinHeader_2.54mm:PinHeader_1x04_P2.54mm_Vertical
- J4, J5: footprint Connector_PinHeader_1.27mm:PinHeader_1x02_P1.27mm_Vertical -> Connector_PinHeader_2.54mm:PinHeader_1x02_P2.54mm_Vertical
Changed lines of the file:
@@
 F 0 "D3" H 8550 4650 50  0000 L CNN
 F 1 "NeoPixel_THT" H 8800 4150 50  0000 L CNN
-F 2 "Connector_PinHeader_1.27mm:PinHeader_1x04_P1.27mm_Vertical" H 8800 4100 50  0001 L TNN
+F 2 "Connector_PinHeader_2.54mm:PinHeader_1x04_P2.54mm_Vertical" H 8800 4100 50  0001 L TNN
 F 3 "https://www.adafruit.com/product/1938" H 8850 4025 50  0001 L TNN
 F 4 "1938" H 0   0   50  0001 C CNN "MPN"
@@
 F 0 "D2" H 7600 4650 50  0000 L CNN
 F 1 "NeoPixel_THT" H 7850 4150 50  0000 L CNN
-F 2 "Connector_PinHeader_1.27mm:PinHeader_1x04_P1.27mm_Vertical" H 7850 4100 50  0001 L TNN
+F 2 "Connector_PinHeader_2.54mm:PinHeader_1x04_P2.54mm_Vertical" H 7850 4100 50  0001 L TNN
 F 3 "https://www.adafruit.com/product/1938" H 7900 4025 50  0001 L TNN
 F 4 "1938" H 0   0   50  0001 C CNN "MPN"
@@
 F 0 "J5" H 5080 1242 50  0000 L CNN
 F 1 "Port_2" H 5080 1151 50  0000 L CNN
-F 2 "Connector_PinHeader_1.27mm:PinHeader_1x02_P1.27mm_Vertical" H 5000 1250 50  0001 C CNN
+F 2 "Connector_PinHeader_2.54mm:PinHeader_1x02_P2.54mm_Vertical" H 5000 1250 50  0001 C CNN
 F 3 "~" H 5000 1250 50  0001 C CNN
 	1    5000 1250
@@
 F 0 "J4" H 5080 792 50  0000 L CNN
 F 1 "Port_1" H 5080 701 50  0000 L CNN
-F 2 "Connector_PinHeader_1.27mm:PinHeader_1x02_P1.27mm_Vertical" H 5000 800 50  0001 C CNN
+F 2 "Connector_PinHeader_2.54mm:PinHeader_1x02_P2.54mm_Vertical" H 5000 800 50  0001 C CNN
 F 3 "~" H 5000 800 50  0001 C CNN
 	1    5000 800

Commit message: Numbered LEDs (values)
Parts:
- D2: value NeoPixel_THT -> LED 1
- D3: value NeoPixel_THT -> LED 2
- U4: symbol top-hemi-rescue:ADXL335-SparkfunSensors -> top-hemi-rescue:ADXL335-SparkfunSensors-top-hemi-rescue
Changed lines of the file:
@@
 AR Path="/5C920754/5C95CBD5" Ref="D3"  Part="1"
 F 0 "D3" H 8550 4650 50  0000 L CNN
-F 1 "NeoPixel_THT" H 8800 4150 50  0000 L CNN
+F 1 "LED 2" H 8800 4150 50  0000 L CNN
 F 2 "Connector_PinHeader_2.54mm:PinHeader_1x04_P2.54mm_Vertical" H 8800 4100 50  0001 L TNN
 F 3 "https://www.adafruit.com/product/1938" H 8850 4025 50  0001 L TNN
@@
 AR Path="/5C920754/5C95CBDB" Ref="D2"  Part="1"
 F 0 "D2" H 7600 4650 50  0000 L CNN
-F 1 "NeoPixel_THT" H 7850 4150 50  0000 L CNN
+F 1 "LED 1" H 7850 4150 50  0000 L CNN
 F 2 "Connector_PinHeader_2.54mm:PinHeader_1x04_P2.54mm_Vertical" H 7850 4100 50  0001 L TNN
 F 3 "https://www.adafruit.com/product/1938" H 7900 4025 50  0001 L TNN
@@
 $EndComp
 $Comp
-L top-hemi-rescue:ADXL335-SparkfunSensors U?
+L top-hemi-rescue:ADXL335-SparkfunSensors-top-hemi-rescue U?
 U 1 1 5C9710AE
 P 8150 3150

Commit message: Connect USB-Mini shield to GND
Connections:
- wire segments 80 -> 81
Changed lines of the file:
@@
 Wire Wire Line
 	1550 3400 2050 3400
+Wire Wire Line
+	1750 5350 1850 5350
+Connection ~ 1850 5350
 $EndSCHEMATC
