File: top.sch (KiCad schematic (older format))
At the start: 27 parts, among them J1 USB_B_Mini, J2 TC2030_NL, J3 FFC-0.5MM-6POS, J4 Port_1, J5 Port_2, U1 PMIC-LDO-XC6204B332MR_SOT23-5_, U2 LP2985-5.0, U3 ATmega328P-MU, U4 ADXL337, Y1 16MHz

Commit message: Connect ST to GND, to be on the safe side
Connections:
- wire segments 80 -> 81
- no-connect marks 3 -> 2
Other:
- note added: "See EVAL-ADXL337Z eval board / UG-242"
- moved on the sheet: C10, C8
Changed lines of the file:
@@
 L power:GND #PWR?
 U 1 1 5C971076
-P 7300 3150
+P 7700 1700
 AR Path="/5C971076" Ref="#PWR?"  Part="1"
 AR Path="/5C920754/5C971076" Ref="#PWR024"  Part="1"
-F 0 "#PWR024" H 7300 2900 50  0001 C CNN
-F 1 "GND" H 7305 2977 50  0000 C CNN
-F 2 "" H 7300 3150 50  0001 C CNN
-F 3 "" H 7300 3150 50  0001 C CNN
-	1    7300 3150
+F 0 "#PWR024" H 7700 1450 50  0001 C CNN
+F 1 "GND" H 7705 1527 50  0000 C CNN
+F 2 "" H 7700 1700 50  0001 C CNN
+F 3 "" H 7700 1700 50  0001 C CNN
+	1    7700 1700
 	1    0    0    -1
 $EndComp
@@
 L power:+3V3 #PWR?
 U 1 1 5C97107C
-P 7300 2950
+P 7700 1500
 AR Path="/5C97107C" Ref="#PWR?"  Part="1"
 AR Path="/5C920754/5C97107C" Ref="#PWR023"  Part="1"
-F 0 "#PWR023" H 7300 2800 50  0001 C CNN
-F 1 "+3V3" H 7315 3123 50  0000 C CNN
-F 2 "" H 7300 2950 50  0001 C CNN
-F 3 "" H 7300 2950 50  0001 C CNN
-	1    7300 2950
+F 0 "#PWR023" H 7700 1350 50  0001 C CNN
+F 1 "+3V3" H 7715 1673 50  0000 C CNN
+F 2 "" H 7700 1500 50  0001 C CNN
+F 3 "" H 7700 1500 50  0001 C CNN
+	1    7700 1500
 	1    0    0    -1
 $EndComp
@@
 L Device:C_Small C?
 U 1 1 5C971082
-P 7300 3050
+P 7700 1600
 AR Path="/5C971082" Ref="C?"  Part="1"
 AR Path="/5C920754/5C971082" Ref="C8"  Part="1"
-F 0 "C8" H 7392 3096 50  0000 L CNN
-F 1 "0.1u" H 7392 3005 50  0000 L CNN
-F 2 "Capacitor_SMD:C_0402_1005Metric" H 7300 3050 50  0001 C CNN
-F 3 "~" H 7300 3050 50  0001 C CNN
-F 4 "VJ0402G104KXQCW1BC" H 0   0   50  0001 C CNN "MPN"
-F 5 "VJ0402G104KXQCW1BC" H 0   0   50  0001 C CNN "SKU"
-F 6 "Shenzhen" H 0   0   50  0001 C CNN "OPL"
-F 7 "50" H 0   0   50  0001 C CNN "Min Quantity"
-	1    7300 3050
+F 0 "C8" H 7792 1646 50  0000 L CNN
+F 1 "0.1u" H 7792 1555 50  0000 L CNN
+F 2 "Capacitor_SMD:C_0402_1005Metric" H 7700 1600 50  0001 C CNN
+F 3 "~" H 7700 1600 50  0001 C CNN
+F 4 "VJ0402G104KXQCW1BC" H 400 -1450 50  0001 C CNN "MPN"
+F 5 "VJ0402G104KXQCW1BC" H 400 -1450 50  0001 C CNN "SKU"
+F 6 "Shenzhen" H 400 -1450 50  0001 C CNN "OPL"
+F 7 "50" H 400 -1450 50  0001 C CNN "Min Quantity"
+	1    7700 1600
 	1    0    0    -1
 $EndComp
@@
 L power:+3V3 #PWR?
 U 1 1 5C97108B
-P 7650 2750
+P 8050 1300
 AR Path="/5C97108B" Ref="#PWR?"  Part="1"
 AR Path="/5C920754/5C97108B" Ref="#PWR025"  Part="1"
-F 0 "#PWR025" H 7650 2600 50  0001 C CNN
-F 1 "+3V3" H 7665 2923 50  0000 C CNN
-F 2 "" H 7650 2750 50  0001 C CNN
-F 3 "" H 7650 2750 50  0001 C CNN
-	1    7650 2750
+F 0 "#PWR025" H 8050 1150 50  0001 C CNN
+F 1 "+3V3" H 8065 1473 50  0000 C CNN
+F 2 "" H 8050 1300 50  0001 C CNN
+F 3 "" H 8050 1300 50  0001 C CNN
+	1    8050 1300
 	1    0    0    -1
 $EndComp
@@
 L power:GND #PWR?
 U 1 1 5C971097
-P 7650 3450
+P 8050 2000
 AR Path="/5C971097" Ref="#PWR?"  Part="1"
 AR Path="/5C920754/5C971097" Ref="#PWR026"  Part="1"
-F 0 "#PWR026" H 7650 3200 50  0001 C CNN
-F 1 "GND" H 7655 3277 50  0000 C CNN
-F 2 "" H 7650 3450 50  0001 C CNN
-F 3 "" H 7650 3450 50  0001 C CNN
-	1    7650 3450
-	1    0    0    -1
-$EndComp
-Connection ~ 8950 3050
-Wire Wire Line
-	9100 3050 8950 3050
+F 0 "#PWR026" H 8050 1750 50  0001 C CNN
+F 1 "GND" H 8055 1827 50  0000 C CNN
+F 2 "" H 8050 2000 50  0001 C CNN
+F 3 "" H 8050 2000 50  0001 C CNN
+	1    8050 2000
+	1    0    0    -1
+$EndComp
+Connection ~ 9350 1600
+Wire Wire Line
+	9500 1600 9350 1600
 $Comp
 L power:GND #PWR?
 U 1 1 5C9710A0
-P 8950 3350
+P 9350 1900
 AR Path="/5C9710A0" Ref="#PWR?"  Part="1"
 AR Path="/5C920754/5C9710A0" Ref="#PWR031"  Part="1"
-F 0 "#PWR031" H 8950 3100 50  0001 C CNN
-F 1 "GND" H 8955 3177 50  0000 C CNN
-F 2 "" H 8950 3350 50  0001 C CNN
-F 3 "" H 8950 3350 50  0001 C CNN
-	1    8950 3350
-	1    0    0    -1
-$EndComp
-Wire Wire Line
-	8950 3050 8950 3150
-Wire Wire Line
-	8650 3050 8950 3050
+F 0 "#PWR031" H 9350 1650 50  0001 C CNN
+F 1 "GND" H 9355 1727 50  0000 C CNN
+F 2 "" H 9350 1900 50  0001 C CNN
+F 3 "" H 9350 1900 50  0001 C CNN
+	1    9350 1900
+	1    0    0    -1
+$EndComp
+Wire Wire Line
+	9350 1600 9350 1700
+Wire Wire Line
+	9050 1600 9350 1600
 $Comp
 L Device:C_Small C?
 U 1 1 5C9710A8
-P 8950 3250
+P 9350 1800
 AR Path="/5C9710A8" Ref="C?"  Part="1"
 AR Path="/5C920754/5C9710A8" Ref="C10"  Part="1"
-F 0 "C10" H 9042 3296 50  0000 L CNN
-F 1 "0.1u" H 9042 3205 50  0000 L CNN
-F 2 "Capacitor_SMD:C_0402_1005Metric" H 8950 3250 50  0001 C CNN
-F 3 "~" H 8950 3250 50  0001 C CNN
-F 4 "VJ0402G104KXQCW1BC" H 0   0   50  0001 C CNN "MPN"
-F 5 "VJ0402G104KXQCW1BC" H 0   0   50  0001 C CNN "SKU"
-F 6 "Shenzhen" H 0   0   50  0001 C CNN "OPL"
-F 7 "50" H 0   0   50  0001 C CNN "Min Quantity"
-	1    8950 3250
+F 0 "C10" H 9442 1846 50  0000 L CNN
+F 1 "0.1u" H 9442 1755 50  0000 L CNN
+F 2 "Capacitor_SMD:C_0402_1005Metric" H 9350 1800 50  0001 C CNN
+F 3 "~" H 9350 1800 50  0001 C CNN
+F 4 "VJ0402G104KXQCW1BC" H 400 -1450 50  0001 C CNN "MPN"
+F 5 "VJ0402G104KXQCW1BC" H 400 -1450 50  0001 C CNN "SKU"
+F 6 "Shenzhen" H 400 -1450 50  0001 C CNN "OPL"
+F 7 "50" H 400 -1450 50  0001 C CNN "Min Quantity"
+	1    9350 1800
 	1    0    0    -1
 $EndComp
@@
 Text Label 4100 6650 0    50   ~ 0
 BNC-3
-Text Label 9100 3050 0    50   ~ 0
+Text Label 9500 1600 0    50   ~ 0
 Z-ACCEL
 Text Label 9350 4400 0    50   ~ 0
@@
 	1900 5350 2000 5350
 Connection ~ 2000 5350
-NoConn ~ 8650 2850
-NoConn ~ 8650 2950
-NoConn ~ 8650 3250
-Wire Wire Line
-	7650 2750 7650 2850
+NoConn ~ 9050 1400
+NoConn ~ 9050 1500
+Wire Wire Line
+	8050 1300 8050 1400
 $Comp
 L SparkFun-Sensors:ADXL337 U4
 U 1 1 5C9C6311
-P 8150 3050
-F 0 "U4" H 8150 3610 45  0000 C CNN
-F 1 "ADXL337" H 8150 3526 45  0000 C CNN
-F 2 "Package_CSP:LFCSP-16-1EP_3x3mm_P0.5mm_EP1.6x1.6mm" H 8150 3450 20  0001 C CNN
-F 3 "" H 8150 3050 60  0001 C CNN
-F 4 "IC-12011" H 8150 3431 60  0000 C CNN "Field4"
-	1    8150 3050
-	1    0    0    -1
-$EndComp
-Wire Wire Line
-	7650 2950 7650 2850
-Connection ~ 7650 2850
-Wire Wire Line
-	7650 3150 7650 3250
-Connection ~ 7650 3250
-Wire Wire Line
-	7650 3250 7650 3450
+P 8550 1600
+F 0 "U4" H 8550 2160 45  0000 C CNN
+F 1 "ADXL337" H 8550 2076 45  0000 C CNN
+F 2 "Package_CSP:LFCSP-16-1EP_3x3mm_P0.5mm_EP1.6x1.6mm" H 8550 2000 20  0001 C CNN
+F 3 "" H 8550 1600 60  0001 C CNN
+F 4 "IC-12011" H 8550 1981 60  0000 C CNN "Field4"
+	1    8550 1600
+	1    0    0    -1
+$EndComp
+Wire Wire Line
+	8050 1500 8050 1400
+Connection ~ 8050 1400
+Wire Wire Line
+	8050 1700 8050 1800
+Connection ~ 8050 1800
+Wire Wire Line
+	8050 1800 8050 2000
+Text Notes 7800 2500 0    50   ~ 0
+See EVAL-ADXL337Z eval board / UG-242
+Wire Notes Line
+	9500 2400 9500 2550
+Wire Notes Line
+	9500 2550 7750 2550
+Wire Notes Line
+	7750 2550 7750 2400
+$Comp
+L power:GND #PWR?
+U 1 1 5C9EBDEA
+P 9050 1900
+AR Path="/5C9EBDEA" Ref="#PWR?"  Part="1"
+AR Path="/5C920754/5C9EBDEA" Ref="#PWR?"  Part="1"
+F 0 "#PWR?" H 9050 1650 50  0001 C CNN
+F 1 "GND" H 9055 1727 50  0000 C CNN
+F 2 "" H 9050 1900 50  0001 C CNN
+F 3 "" H 9050 1900 50  0001 C CNN
+	1    9050 1900
+	1    0    0    -1
+$EndComp
+Wire Wire Line
+	9050 1900 9050 1800
+Wire Notes Line
+	7750 2400 9500 2400
 $EndSCHEMATC

Commit message: Revice voltage regulator circuits
Parts:
- added C14: 1u, Capacitor_SMD:C_0603_1608Metric, symbol Device:C_Small
Connections:
- wire segments 81 -> 88
- no-connect marks 2 -> 4
Other:
- note added: "See LP2985-N datasheet ([0.01uF \ncapacitor on BP] may be omitted\nif application is not noise critical)"
- note added: "See XC6204/XC6205 datasheet\n("Please wire the input capacitor (CIN)\nand the output capacitor (CL) as close\nto the IC as possible.")"
- moved on the sheet: BT1, C1, C2, C3, C4, D1, J1, J2, U1, U2

Commit message: Switch to WS2812D-F5 (NeoPixel w/ diff. pinout)
Parts:
- removed D2: LED 1, node:WS2812D-F5, symbol LED:NeoPixel_THT
- removed D3: LED 2, node:WS2812D-F5, symbol LED:NeoPixel_THT
- added D2, D3: WS2812D-F5, node:WS2812D-F5, symbol node:WS2812D-F5
Other:
- moved on the sheet: C11, C9
Changed lines of the file:
@@
 L power:+5V #PWR?
 U 1 1 5C95CB94
-P 7800 3950
+P 8025 4050
 AR Path="/5C95CB94" Ref="#PWR?"  Part="1"
 AR Path="/5C920754/5C95CB94" Ref="#PWR027"  Part="1"
-F 0 "#PWR027" H 7800 3800 50  0001 C CNN
-F 1 "+5V" H 7815 4123 50  0000 C CNN
-F 2 "" H 7800 3950 50  0001 C CNN
-F 3 "" H 7800 3950 50  0001 C CNN
-	1    7800 3950
+F 0 "#PWR027" H 8025 3900 50  0001 C CNN
+F 1 "+5V" H 8040 4223 50  0000 C CNN
+F 2 "" H 8025 4050 50  0001 C CNN
+F 3 "" H 8025 4050 50  0001 C CNN
+	1    8025 4050
 	1    0    0    -1
 $EndComp
@@
 L power:+5V #PWR?
 U 1 1 5C95CB9A
-P 8750 3950
+P 9400 4050
 AR Path="/5C95CB9A" Ref="#PWR?"  Part="1"
 AR Path="/5C920754/5C95CB9A" Ref="#PWR029"  Part="1"
-F 0 "#PWR029" H 8750 3800 50  0001 C CNN
-F 1 "+5V" H 8765 4123 50  0000 C CNN
-F 2 "" H 8750 3950 50  0001 C CNN
-F 3 "" H 8750 3950 50  0001 C CNN
-	1    8750 3950
+F 0 "#PWR029" H 9400 3900 50  0001 C CNN
+F 1 "+5V" H 9415 4223 50  0000 C CNN
+F 2 "" H 9400 4050 50  0001 C CNN
+F 3 "" H 9400 4050 50  0001 C CNN
+	1    9400 4050
 	1    0    0    -1
 $EndComp
@@
 L Device:C_Small C?
 U 1 1 5C95CBA0
-P 8150 4150
+P 8650 4250
 AR Path="/5C95CBA0" Ref="C?"  Part="1"
 AR Path="/5C920754/5C95CBA0" Ref="C9"  Part="1"
-F 0 "C9" H 8242 4196 50  0000 L CNN
-F 1 "0.1u" H 8242 4105 50  0000 L CNN
-F 2 "Capacitor_SMD:C_0402_1005Metric" H 8150 4150 50  0001 C CNN
-F 3 "~" H 8150 4150 50  0001 C CNN
-F 4 "VJ0402G104KXQCW1BC" H 0   0   50  0001 C CNN "MPN"
-F 5 "VJ0402G104KXQCW1BC" H 0   0   50  0001 C CNN "SKU"
-F 6 "Shenzhen" H 0   0   50  0001 C CNN "OPL"
-F 7 "50" H 0   0   50  0001 C CNN "Min Quantity"
-	1    8150 4150
+F 0 "C9" H 8742 4296 50  0000 L CNN
+F 1 "0.1u" H 8742 4205 50  0000 L CNN
+F 2 "Capacitor_SMD:C_0402_1005Metric" H 8650 4250 50  0001 C CNN
+F 3 "~" H 8650 4250 50  0001 C CNN
+F 4 "VJ0402G104KXQCW1BC" H 500 100 50  0001 C CNN "MPN"
+F 5 "VJ0402G104KXQCW1BC" H 500 100 50  0001 C CNN "SKU"
+F 6 "Shenzhen" H 500 100 50  0001 C CNN "OPL"
+F 7 "50" H 500 100 50  0001 C CNN "Min Quantity"
+	1    8650 4250
 	1    0    0    -1
 $EndComp
@@
 L Device:C_Small C?
 U 1 1 5C95CBA6
-P 9100 4150
+P 10025 4250
 AR Path="/5C95CBA6" Ref="C?"  Part="1"
 AR Path="/5C920754/5C95CBA6" Ref="C11"  Part="1"
-F 0 "C11" H 9192 4196 50  0000 L CNN
-F 1 "0.1u" H 9192 4105 50  0000 L CNN
-F 2 "Capacitor_SMD:C_0402_1005Metric" H 9100 4150 50  0001 C CNN
-F 3 "~" H 9100 4150 50  0001 C CNN
-F 4 "VJ0402G104KXQCW1BC" H 0   0   50  0001 C CNN "MPN"
-F 5 "VJ0402G104KXQCW1BC" H 0   0   50  0001 C CNN "SKU"
-F 6 "Shenzhen" H 0   0   50  0001 C CNN "OPL"
-F 7 "50" H 0   0   50  0001 C CNN "Min Quantity"
-	1    9100 4150
-	1    0    0    -1
-$EndComp
-Wire Wire Line
-	9350 4400 9050 4400
-Wire Wire Line
-	7400 4400 7500 4400
+F 0 "C11" H 10117 4296 50  0000 L CNN
+F 1 "0.1u" H 10117 4205 50  0000 L CNN
+F 2 "Capacitor_SMD:C_0402_1005Metric" H 10025 4250 50  0001 C CNN
+F 3 "~" H 10025 4250 50  0001 C CNN
+F 4 "VJ0402G104KXQCW1BC" H 925 100 50  0001 C CNN "MPN"
+F 5 "VJ0402G104KXQCW1BC" H 925 100 50  0001 C CNN "SKU"
+F 6 "Shenzhen" H 925 100 50  0001 C CNN "OPL"
+F 7 "50" H 925 100 50  0001 C CNN "Min Quantity"
+	1    10025 4250
+	1    0    0    -1
+$EndComp
+Wire Wire Line
+	7625 4500 7725 4500
 $Comp
 L power:GND #PWR?
 U 1 1 5C95CBC8
-P 8750 4800
+P 9400 4900
 AR Path="/5C95CBC8" Ref="#PWR?"  Part="1"
 AR Path="/5C920754/5C95CBC8" Ref="#PWR030"  Part="1"
-F 0 "#PWR030" H 8750 4550 50  0001 C CNN
-F 1 "GND" H 8755 4627 50  0000 C CNN
-F 2 "" H 8750 4800 50  0001 C CNN
-F 3 "" H 8750 4800 50  0001 C CNN
-	1    8750 4800
+F 0 "#PWR030" H 9400 4650 50  0001 C CNN
+F 1 "GND" H 9405 4727 50  0000 C CNN
+F 2 "" H 9400 4900 50  0001 C CNN
+F 3 "" H 9400 4900 50  0001 C CNN
+	1    9400 4900
 	1    0    0    -1
 $EndComp
@@
 L power:GND #PWR?
 U 1 1 5C95CBCE
-P 7800 4800
+P 8025 4900
 AR Path="/5C95CBCE" Ref="#PWR?"  Part="1"
 AR Path="/5C920754/5C95CBCE" Ref="#PWR028"  Part="1"
-F 0 "#PWR028" H 7800 4550 50  0001 C CNN
-F 1 "GND" H 7805 4627 50  0000 C CNN
-F 2 "" H 7800 4800 50  0001 C CNN
-F 3 "" H 7800 4800 50  0001 C CNN
-	1    7800 4800
-	1    0    0    -1
-$EndComp
-Wire Wire Line
-	8100 4400 8450 4400
-$Comp
-L LED:NeoPixel_THT D?
-U 1 1 5C95CBD5
-P 8750 4400
-AR Path="/5C95CBD5" Ref="D?"  Part="1"
-AR Path="/5C920754/5C95CBD5" Ref="D3"  Part="1"
-F 0 "D3" H 8550 4650 50  0000 L CNN
-F 1 "LED 2" H 8800 4150 50  0000 L CNN
-F 2 "node:WS2812D-F5" H 8800 4100 50  0001 L TNN
-F 3 "https://www.adafruit.com/product/1938" H 8850 4025 50  0001 L TNN
-F 4 "1938" H 0   0   50  0001 C CNN "MPN"
-F 5 "1528-1959-ND	" H 0   0   50  0001 C CNN "SKU"
-F 6 "5" H 0   0   50  0001 C CNN "Min Quantity"
-	1    8750 4400
-	1    0    0    -1
-$EndComp
-$Comp
-L LED:NeoPixel_THT D?
-U 1 1 5C95CBDB
-P 7800 4400
-AR Path="/5C95CBDB" Ref="D?"  Part="1"
-AR Path="/5C920754/5C95CBDB" Ref="D2"  Part="1"
-F 0 "D2" H 7600 4650 50  0000 L CNN
-F 1 "LED 1" H 7850 4150 50  0000 L CNN
-F 2 "node:WS2812D-F5" H 7850 4100 50  0001 L TNN
-F 3 "https://www.adafruit.com/product/1938" H 7900 4025 50  0001 L TNN
-F 4 "1938" H 0   0   50  0001 C CNN "MPN"
-F 5 "1528-1959-ND	" H 0   0   50  0001 C CNN "SKU"
-F 6 "5" H 0   0   50  0001 C CNN "Min Quantity"
-	1    7800 4400
-	1    0    0    -1
-$EndComp
-Wire Wire Line
-	7800 3950 7800 4050
-Wire Wire Line
-	7800 4050 8150 4050
-Connection ~ 7800 4050
-Wire Wire Line
-	7800 4050 7800 4100
-Wire Wire Line
-	7800 4750 8150 4750
-Wire Wire Line
-	8150 4750 8150 4250
-Wire Wire Line
-	7800 4700 7800 4750
-Connection ~ 7800 4750
-Wire Wire Line
-	7800 4750 7800 4800
-Wire Wire Line
-	8750 4100 8750 4050
-Wire Wire Line
-	8750 4050 9100 4050
-Connection ~ 8750 4050
-Wire Wire Line
-	8750 4050 8750 3950
-Wire Wire Line
-	8750 4800 8750 4750
-Wire Wire Line
-	8750 4750 9100 4750
-Wire Wire Line
-	9100 4750 9100 4250
-Connection ~ 8750 4750
-Wire Wire Line
-	8750 4750 8750 4700
+F 0 "#PWR028" H 8025 4650 50  0001 C CNN
+F 1 "GND" H 8030 4727 50  0000 C CNN
+F 2 "" H 8025 4900 50  0001 C CNN
+F 3 "" H 8025 4900 50  0001 C CNN
+	1    8025 4900
+	1    0    0    -1
+$EndComp
+Wire Wire Line
+	8325 4500 9100 4500
+Wire Wire Line
+	8025 4050 8025 4150
+Wire Wire Line
+	8025 4150 8650 4150
+Connection ~ 8025 4150
+Wire Wire Line
+	8025 4150 8025 4200
+Wire Wire Line
+	8025 4850 8650 4850
+Wire Wire Line
+	8650 4850 8650 4350
+Wire Wire Line
+	8025 4800 8025 4850
+Connection ~ 8025 4850
+Wire Wire Line
+	8025 4850 8025 4900
+Wire Wire Line
+	9400 4200 9400 4150
+Wire Wire Line
+	9400 4150 10025 4150
+Connection ~ 9400 4150
+Wire Wire Line
+	9400 4150 9400 4050
+Wire Wire Line
+	9400 4900 9400 4850
+Wire Wire Line
+	9400 4850 10025 4850
+Wire Wire Line
+	10025 4850 10025 4350
+Connection ~ 9400 4850
+Wire Wire Line
+	9400 4850 9400 4800
 Text Label 6100 4500 0    50   ~ 0
 DIN-TOP
-Text Label 7400 4400 2    50   ~ 0
+Text Label 7625 4500 2    50   ~ 0
 DIN-TOP
 $Comp
@@
 Text Label 9500 1600 0    50   ~ 0
 Z-ACCEL
-Text Label 9350 4400 0    50   ~ 0
+Text Label 10275 4500 0    50   ~ 0
 DOUT-BOT
 Text Label 4100 6850 0    50   ~ 0
@@
 Wire Wire Line
 	8050 1800 8050 2000
-Text Notes 7795 2513 0    50   ~ 0
+Text Notes 7795 2413 0    50   ~ 0
 See EVAL-ADXL337Z eval board / UG-242
 Wire Notes Line
-	9500 2400 9500 2550
-Wire Notes Line
-	9500 2550 7750 2550
-Wire Notes Line
-	7750 2550 7750 2400
+	9500 2300 9500 2450
+Wire Notes Line
+	9500 2450 7750 2450
+Wire Notes Line
+	7750 2450 7750 2300
 $Comp
 L power:GND #PWR?
@@
 	9050 1900 9050 1800
 Wire Notes Line
-	7750 2400 9500 2400
+	7750 2300 9500 2300
 $Comp
 L SparkFun-Sensors:ADXL337 U4
@@
 Wire Notes Line
 	1350 3425 1350 3100
+$Comp
+L node:WS2812D-F5 D2
+U 1 1 5C98F418
+P 8025 4500
+F 0 "D2" H 7825 4750 50  0000 L CNN
+F 1 "WS2812D-F5" H 8050 4250 50  0000 L CNN
+F 2 "node:WS2812D-F5" H 8075 4200 50  0001 L TNN
+F 3 "http://www.world-semi.com/DownLoadFile/135" H 8125 4125 50  0001 L TNN
+	1    8025 4500
+	1    0    0    -1
+$EndComp
+$Comp
+L node:WS2812D-F5 D3
+U 1 1 5C993699
+P 9400 4500
+F 0 "D3" H 9200 4750 50  0000 L CNN
+F 1 "WS2812D-F5" H 9450 4250 50  0000 L CNN
+F 2 "node:WS2812D-F5" H 9450 4200 50  0001 L TNN
+F 3 "http://www.world-semi.com/DownLoadFile/135" H 9500 4125 50  0001 L TNN
+	1    9400 4500
+	1    0    0    -1
+$EndComp
+Wire Wire Line
+	9700 4500 10275 4500
 $EndSCHEMATC

Commit message: Add PicoBlade connectors
Parts:
- J4, J5: footprint node:port -> Connector_Molex:Molex_PicoBlade_53047-0210_1x02_P1.25mm_Vertical
Changed lines of the file:
@@
 F 0 "J5" H 5080 1242 50  0000 L CNN
 F 1 "Port_2" H 5080 1151 50  0000 L CNN
-F 2 "node:port" H 5000 1250 50  0001 C CNN
+F 2 "Connector_Molex:Molex_PicoBlade_53047-0210_1x02_P1.25mm_Vertical" H 5000 1250 50  0001 C CNN
 F 3 "~" H 5000 1250 50  0001 C CNN
 	1    5000 1250
@@
 F 0 "J4" H 5080 792 50  0000 L CNN
 F 1 "Port_1" H 5080 701 50  0000 L CNN
-F 2 "node:port" H 5000 800 50  0001 C CNN
+F 2 "Connector_Molex:Molex_PicoBlade_53047-0210_1x02_P1.25mm_Vertical" H 5000 800 50  0001 C CNN
 F 3 "~" H 5000 800 50  0001 C CNN
 	1    5000 800

Commit message: Configure ADXL337 pins to avoid ERC warnings
Parts:
- removed U4: ADXL337, Package_CSP:LFCSP-16-1EP_3x3mm_P0.5mm_EP1.6x1.6mm, symbol SparkFun-Sensors:ADXL337
- added U4: ADXL337, LFCSP-16-3X3, symbol node:ADXL337
Connections:
- no-connect marks 4 -> 15
Changed lines of the file:
@@
 L power:GND #PWR?
 U 1 1 5C9566B1
-P 1250 4600
+P 1250 4650
 AR Path="/5C9566B1" Ref="#PWR?"  Part="1"
 AR Path="/5C920754/5C9566B1" Ref="#PWR01"  Part="1"
-F 0 "#PWR01" H 1250 4350 50  0001 C CNN
-F 1 "GND" H 1255 4427 50  0000 C CNN
-F 2 "" H 1250 4600 50  0001 C CNN
-F 3 "" H 1250 4600 50  0001 C CNN
-	1    1250 4600
+F 0 "#PWR01" H 1250 4400 50  0001 C CNN
+F 1 "GND" H 1255 4477 50  0000 C CNN
+F 2 "" H 1250 4650 50  0001 C CNN
+F 3 "" H 1250 4650 50  0001 C CNN
+	1    1250 4650
 	1    0    0    -1
 $EndComp
@@
 F 3 "" H 2850 2400 50  0001 C CNN
 	1    2850 2400
-	1    0    0    -1
-$EndComp
-$Comp
-L power:GND #PWR?
-U 1 1 5C9566C3
-P 1950 4600
-AR Path="/5C9566C3" Ref="#PWR?"  Part="1"
-AR Path="/5C920754/5C9566C3" Ref="#PWR05"  Part="1"
-F 0 "#PWR05" H 1950 4350 50  0001 C CNN
-F 1 "GND" H 1955 4427 50  0000 C CNN
-F 2 "" H 1950 4600 50  0001 C CNN
-F 3 "" H 1950 4600 50  0001 C CNN
-	1    1950 4600
 	1    0    0    -1
 $EndComp
@@
 NoConn ~ 9050 1400
 NoConn ~ 9050 1500
-Wire Wire Line
-	8050 1300 8050 1400
-Wire Wire Line
-	8050 1500 8050 1400
-Connection ~ 8050 1400
-Wire Wire Line
-	8050 1700 8050 1800
-Connection ~ 8050 1800
-Wire Wire Line
-	8050 1800 8050 2000
 Text Notes 7795 2413 0    50   ~ 0
 See EVAL-ADXL337Z eval board / UG-242
@@
 Wire Notes Line
 	7750 2300 9500 2300
-$Comp
-L SparkFun-Sensors:ADXL337 U4
-U 1 1 5C9C6311
-P 8550 1600
-F 0 "U4" H 8550 2160 45  0000 C CNN
-F 1 "ADXL337" H 8550 2076 45  0000 C CNN
-F 2 "Package_CSP:LFCSP-16-1EP_3x3mm_P0.5mm_EP1.6x1.6mm" H 8550 2000 20  0001 C CNN
-F 3 "" H 8550 1600 60  0001 C CNN
-F 4 "IC-12011" H 8550 1981 60  0000 C CNN "Field4"
-	1    8550 1600
-	1    0    0    -1
-$EndComp
 $Comp
 L Device:C_Small C?
@@
 See LP2985-N datasheet ([0.01uF \ncapacitor on BP]  may be omitted\nif application is not noise critical)
 Connection ~ 2850 2400
-Text Notes 1250 5250 0    50   ~ 0
+Text Notes 1250 5300 0    50   ~ 0
 See XC6204/XC6205 datasheet\n("Please wire the input capacitor (CIN)\nand the output capacitor (CL) as close\nto the IC as possible.")
 Wire Notes Line
-	1200 4900 2800 4900
-Wire Notes Line
-	2800 4900 2800 5300
-Wire Notes Line
-	2800 5300 1200 5300
-Wire Notes Line
-	1200 5300 1200 4900
+	1200 4950 2800 4950
+Wire Notes Line
+	2800 4950 2800 5350
+Wire Notes Line
+	2800 5350 1200 5350
+Wire Notes Line
+	1200 5350 1200 4950
 $Comp
 L Device:C_Small C?
@@
 L power:GND #PWR?
 U 1 1 5C9566AB
-P 2725 4600
+P 2725 4650
 AR Path="/5C9566AB" Ref="#PWR?"  Part="1"
 AR Path="/5C920754/5C9566AB" Ref="#PWR010"  Part="1"
-F 0 "#PWR010" H 2725 4350 50  0001 C CNN
-F 1 "GND" H 2730 4427 50  0000 C CNN
-F 2 "" H 2725 4600 50  0001 C CNN
-F 3 "" H 2725 4600 50  0001 C CNN
-	1    2725 4600
-	1    0    0    -1
-$EndComp
-Wire Wire Line
-	2725 4600 2725 4475
+F 0 "#PWR010" H 2725 4400 50  0001 C CNN
+F 1 "GND" H 2730 4477 50  0000 C CNN
+F 2 "" H 2725 4650 50  0001 C CNN
+F 3 "" H 2725 4650 50  0001 C CNN
+	1    2725 4650
+	1    0    0    -1
+$EndComp
+Wire Wire Line
+	2725 4650 2725 4475
 Wire Wire Line
 	2725 4100 2725 4125
@@
 	2725 4125 2725 4275
 NoConn ~ 2350 4325
-Wire Wire Line
-	1950 4600 1950 4575
 $Comp
 L OPL_Integrated_Circuit:PMIC-LDO-XC6204B332MR_SOT23-5_ U?
@@
 	1475 4125 1250 4125
 Wire Wire Line
-	1250 4475 1250 4600
+	1250 4475 1250 4650
 Text Label 1250 4125 0    50   ~ 0
 VIN
@@
 Wire Wire Line
 	9700 4500 10275 4500
+$Comp
+L power:GND #PWR?
+U 1 1 5C9566C3
+P 1950 4650
+AR Path="/5C9566C3" Ref="#PWR?"  Part="1"
+AR Path="/5C920754/5C9566C3" Ref="#PWR05"  Part="1"
+F 0 "#PWR05" H 1950 4400 50  0001 C CNN
+F 1 "GND" H 1955 4477 50  0000 C CNN
+F 2 "" H 1950 4650 50  0001 C CNN
+F 3 "" H 1950 4650 50  0001 C CNN
+	1    1950 4650
+	1    0    0    -1
+$EndComp
+Wire Wire Line
+	1950 4650 1950 4575
+Wire Wire Line
+	8050 1800 8050 2000
+Wire Wire Line
+	8050 1700 8050 1800
+Connection ~ 8050 1800
+Wire Wire Line
+	8050 1500 8050 1400
+Wire Wire Line
+	8050 1300 8050 1400
+Connection ~ 8050 1400
+$Comp
+L node:ADXL337 U4
+U 1 1 5C9E1293
+P 8550 1600
+F 0 "U4" H 8200 1950 45  0000 C CNN
+F 1 "ADXL337" H 8800 1250 45  0000 C CNN
+F 2 "LFCSP-16-3X3" H 8550 2000 20  0001 C CNN
+F 3 "" H 8550 1600 60  0001 C CNN
+	1    8550 1600
+	1    0    0    -1
+$EndComp
+NoConn ~ 5200 2600
+NoConn ~ 5200 3400
+NoConn ~ 5200 3500
+NoConn ~ 5200 3600
+NoConn ~ 5200 3700
+NoConn ~ 5200 3800
+NoConn ~ 5200 4600
+NoConn ~ 5200 4700
+NoConn ~ 5200 4800
+NoConn ~ 4000 2600
+NoConn ~ 4000 2675
 $EndSCHEMATC
