File: nodes/pcb/node/node.kicad_pcb (KiCad board)
At the start: 2 copper layers, 46 x 38 mm, 39 parts, among them J1 USB_B_Mini, J2 TC2030_NL, J3 FFC-0.5MM-6POS, J4 Port_1, J5 Port_2, J6 FFC-0.5MM-6POS, J7 Port_3, J8 Port_4, U1 PMIC-LDO-XC6204B332MR_SOT23-5, U2 LP2985-5.0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

Commit message: Add data for assembly drawing file (on F.Fab)
Parts:
- U1: value PMIC-LDO-XC6204B332MR_SOT23-5 -> XC6204B332MR
- U3: value ATmega328P-MU -> 328P-MU
