File: hardware/life_size/nodes/components/main_pcb/kicad/board.sch (KiCad schematic (older format))
At the start: 18 parts

Commit message: Add connector, update numbering
Parts:
- added J8: Power, symbol Connector_Generic:Conn_01x02
- J1: renamed from Port1; value Conn_01x03 -> Port
- J2: renamed from Port2; value Conn_01x03 -> Port
- J3: renamed from Port3; value Conn_01x03 -> Port
- J4: renamed from Port4; value Conn_01x03 -> Port
- J5: renamed from Neopixels; value Conn_01x03 -> Neopixels
- J6: renamed from ESP-EYE; value Conn_01x06 -> ESP-EYE
- J7: renamed from J?; value Conn_01x02 -> Power
- gave numbers to parts that had none: 11
Changed lines of the file:
@@
 $EndDescr
 $Comp
-L SparkFun-Boards:ARDUINO_PRO_MINI B?
+L SparkFun-Boards:ARDUINO_PRO_MINI B1
 U 1 1 5DD15878
 P 2300 2800
-F 0 "B?" H 2300 3754 45  0000 C CNN
+F 0 "B1" H 2300 3754 45  0000 C CNN
 F 1 "ARDUINO_PRO_MINI" H 2300 3670 45  0000 C CNN
 F 2 "ARDUINO_PRO_MINI" H 2300 3750 20  0001 C CNN
@@
 $EndComp
 $Comp
-L power:GND #PWR?
+L power:GND #PWR0101
 U 1 1 5DD1EFE2
 P 975 2625
-F 0 "#PWR?" H 975 2375 50  0001 C CNN
+F 0 "#PWR0101" H 975 2375 50  0001 C CNN
 F 1 "GND" H 980 2452 50  0000 C CNN
 F 2 "" H 975 2625 50  0001 C CNN
@@
 $EndComp
 $Comp
-L Connector_Generic:Conn_01x03 Port4
+L Connector_Generic:Conn_01x03 J4
 U 1 1 5DD282FD
 P 4825 4350
-F 0 "Port4" H 4905 4392 50  0000 L CNN
-F 1 "Conn_01x03" H 4905 4301 50  0000 L CNN
+F 0 "J4" H 4905 4392 50  0000 L CNN
+F 1 "Port" H 4905 4301 50  0000 L CNN
 F 2 "" H 4825 4350 50  0001 C CNN
 F 3 "~" H 4825 4350 50  0001 C CNN
@@
 $EndComp
 $Comp
-L Connector_Generic:Conn_01x03 Port3
+L Connector_Generic:Conn_01x03 J3
 U 1 1 5DD28E2E
 P 4825 4825
-F 0 "Port3" H 4905 4867 50  0000 L CNN
-F 1 "Conn_01x03" H 4905 4776 50  0000 L CNN
+F 0 "J3" H 4905 4867 50  0000 L CNN
+F 1 "Port" H 4905 4776 50  0000 L CNN
 F 2 "" H 4825 4825 50  0001 C CNN
 F 3 "~" H 4825 4825 50  0001 C CNN
@@
 $EndComp
 $Comp
-L Connector_Generic:Conn_01x03 Port2
+L Connector_Generic:Conn_01x03 J2
 U 1 1 5DD2916A
 P 4825 5275
-F 0 "Port2" H 4905 5317 50  0000 L CNN
-F 1 "Conn_01x03" H 4905 5226 50  0000 L CNN
+F 0 "J2" H 4905 5317 50  0000 L CNN
+F 1 "Port" H 4905 5226 50  0000 L CNN
 F 2 "" H 4825 5275 50  0001 C CNN
 F 3 "~" H 4825 5275 50  0001 C CNN
@@
 $EndComp
 $Comp
-L Connector_Generic:Conn_01x03 Port1
+L Connector_Generic:Conn_01x03 J1
 U 1 1 5DD2997A
 P 4825 5700
-F 0 "Port1" H 4905 5742 50  0000 L CNN
-F 1 "Conn_01x03" H 4905 5651 50  0000 L CNN
+F 0 "J1" H 4905 5742 50  0000 L CNN
+F 1 "Port" H 4905 5651 50  0000 L CNN
 F 2 "" H 4825 5700 50  0001 C CNN
 F 3 "~" H 4825 5700 50  0001 C CNN
@@
 $EndComp
 $Comp
-L Device:R_Small_US R?
+L Device:R_Small_US R5
 U 1 1 5DD29F2D
 P 8350 3425
-F 0 "R?" H 8325 3325 50  0000 R CNN
+F 0 "R5" H 8325 3325 50  0000 R CNN
 F 1 "1.7k" H 8325 3525 50  0000 R CNN
 F 2 "" H 8350 3425 50  0001 C CNN
@@
 $EndComp
 $Comp
-L Connector_Generic:Conn_01x06 ESP-EYE
+L Connector_Generic:Conn_01x06 J6
 U 1 1 5DD2B3B7
 P 10400 3650
-F 0 "ESP-EYE" H 10480 3642 50  0000 L CNN
-F 1 "Conn_01x06" H 10480 3551 50  0000 L CNN
+F 0 "J6" H 10480 3642 50  0000 L CNN
+F 1 "ESP-EYE" H 10480 3551 50  0000 L CNN
 F 2 "" H 10400 3650 50  0001 C CNN
 F 3 "~" H 10400 3650 50  0001 C CNN
@@
 $EndComp
 $Comp
-L Connector_Generic:Conn_01x02 J?
+L Connector_Generic:Conn_01x02 J7
 U 1 1 5DD2BB76
 P 5475 1500
-F 0 "J?" H 5555 1492 50  0000 L CNN
-F 1 "Conn_01x02" H 5555 1401 50  0000 L CNN
+F 0 "J7" H 5555 1492 50  0000 L CNN
+F 1 "Power" H 5555 1401 50  0000 L CNN
 F 2 "" H 5475 1500 50  0001 C CNN
 F 3 "~" H 5475 1500 50  0001 C CNN
@@
 $EndComp
 $Comp
-L power:+5V #PWR?
+L power:+5V #PWR0102
 U 1 1 5DD2A9D0
 P 2900 2375
-F 0 "#PWR?" H 2900 2225 50  0001 C CNN
+F 0 "#PWR0102" H 2900 2225 50  0001 C CNN
 F 1 "+5V" H 3025 2425 50  0000 C CNN
 F 2 "" H 2900 2375 50  0001 C CNN
@@
 	2900 2400 2750 2400
 $Comp
-L power:GND #PWR?
+L power:GND #PWR0103
 U 1 1 5DD3224E
 P 3225 2300
-F 0 "#PWR?" H 3225 2050 50  0001 C CNN
+F 0 "#PWR0103" H 3225 2050 50  0001 C CNN
 F 1 "GND" H 3375 2225 50  0000 C CNN
 F 2 "" H 3225 2300 50  0001 C CNN
@@
 	4500 5700 4500 6000
 $Comp
-L power:GND #PWR?
+L power:GND #PWR0104
 U 1 1 5DD34B8B
 P 4500 6000
-F 0 "#PWR?" H 4500 5750 50  0001 C CNN
+F 0 "#PWR0104" H 4500 5750 50  0001 C CNN
 F 1 "GND" H 4505 5827 50  0000 C CNN
 F 2 "" H 4500 6000 50  0001 C CNN
@@
 	1600 4250 4625 4250
 $Comp
-L Connector_Generic:Conn_01x03 Neopixels
+L Connector_Generic:Conn_01x03 J5
 U 1 1 5DD52EAB
 P 6775 3875
-F 0 "Neopixels" H 6855 3917 50  0000 L CNN
-F 1 "Conn_01x03" H 6855 3826 50  0000 L CNN
+F 0 "J5" H 6855 3917 50  0000 L CNN
+F 1 "Neopixels" H 6855 3826 50  0000 L CNN
 F 2 "" H 6775 3875 50  0001 C CNN
 F 3 "~" H 6775 3875 50  0001 C CNN
@@
 $EndComp
 $Comp
-L power:GND #PWR?
+L power:GND #PWR0105
 U 1 1 5DD53728
 P 6475 4150
-F 0 "#PWR?" H 6475 3900 50  0001 C CNN
+F 0 "#PWR0105" H 6475 3900 50  0001 C CNN
 F 1 "GND" H 6625 4075 50  0000 C CNN
 F 2 "" H 6475 4150 50  0001 C CNN
@@
 	6475 3875 6475 4150
 $Comp
-L power:+5V #PWR?
+L power:+5V #PWR0106
 U 1 1 5DD5583D
 P 6350 3650
-F 0 "#PWR?" H 6350 3500 50  0001 C CNN
+F 0 "#PWR0106" H 6350 3500 50  0001 C CNN
 F 1 "+5V" H 6225 3700 50  0000 C CNN
 F 2 "" H 6350 3650 50  0001 C CNN
@@
 	1700 3775 6575 3775
 $Comp
-L power:+5V #PWR?
+L power:+5V #PWR0107
 U 1 1 5DD62987
 P 9750 3300
-F 0 "#PWR?" H 9750 3150 50  0001 C CNN
+F 0 "#PWR0107" H 9750 3150 50  0001 C CNN
 F 1 "+5V" H 9875 3350 50  0000 C CNN
 F 2 "" H 9750 3300 50  0001 C CNN
@@
 	9750 3300 9750 3450
 $Comp
-L power:GND #PWR?
+L power:GND #PWR0108
 U 1 1 5DD647B8
 P 9750 4700
-F 0 "#PWR?" H 9750 4450 50  0001 C CNN
+F 0 "#PWR0108" H 9750 4450 50  0001 C CNN
 F 1 "GND" H 9900 4625 50  0000 C CNN
 F 2 "" H 9750 4700 50  0001 C CNN
@@
 	8350 3200 8350 3325
 $Comp
-L Device:R_Small_US R?
+L Device:R_Small_US R6
 U 1 1 5DD78F8D
 P 8350 4250
-F 0 "R?" H 8325 4150 50  0000 R CNN
+F 0 "R6" H 8325 4150 50  0000 R CNN
 F 1 "3.3k" H 8325 4350 50  0000 R CNN
 F 2 "" H 8350 4250 50  0001 C CNN
@@
 	9100 2900 9100 3325
 $Comp
-L Device:R_Small_US R?
+L Device:R_Small_US R7
 U 1 1 5DD8C49F
 P 8725 3425
-F 0 "R?" H 8700 3325 50  0000 R CNN
+F 0 "R7" H 8700 3325 50  0000 R CNN
 F 1 "1.7k" H 8700 3525 50  0000 R CNN
 F 2 "" H 8725 3425 50  0001 C CNN
@@
 $EndComp
 $Comp
-L Device:R_Small_US R?
+L Device:R_Small_US R9
 U 1 1 5DD8C79E
 P 9100 3425
-F 0 "R?" H 9075 3325 50  0000 R CNN
+F 0 "R9" H 9075 3325 50  0000 R CNN
 F 1 "1.7k" H 9075 3525 50  0000 R CNN
 F 2 "" H 9100 3425 50  0001 C CNN
@@
 $EndComp
 $Comp
-L Device:R_Small_US R?
+L Device:R_Small_US R8
 U 1 1 5DD92DEF
 P 8725 4250
-F 0 "R?" H 8700 4150 50  0000 R CNN
+F 0 "R8" H 8700 4150 50  0000 R CNN
 F 1 "3.3k" H 8700 4350 50  0000 R CNN
 F 2 "" H 8725 4250 50  0001 C CNN
@@
 $EndComp
 $Comp
-L Device:R_Small_US R?
+L Device:R_Small_US R10
 U 1 1 5DD93275
 P 9100 4250
-F 0 "R?" H 9075 4150 50  0000 R CNN
+F 0 "R10" H 9075 4150 50  0000 R CNN
 F 1 "3.3k" H 9075 4350 50  0000 R CNN
 F 2 "" H 9100 4250 50  0001 C CNN
@@
 	9100 3750 9100 4150
 $Comp
-L Device:R_Small_US R?
+L Device:R_Small_US R1
 U 1 1 5DD0D9EE
 P 3200 3500
-F 0 "R?" H 3175 3400 50  0000 R CNN
+F 0 "R1" H 3175 3400 50  0000 R CNN
 F 1 "1k" H 3175 3600 50  0000 R CNN
 F 2 "" H 3200 3500 50  0001 C CNN
@@
 	3200 3600 3200 5800
 $Comp
-L Device:R_Small_US R?
+L Device:R_Small_US R2
 U 1 1 5DD2E8C5
 P 3475 3500
-F 0 "R?" H 3450 3400 50  0000 R CNN
+F 0 "R2" H 3450 3400 50  0000 R CNN
 F 1 "1k" H 3450 3600 50  0000 R CNN
 F 2 "" H 3475 3500 50  0001 C CNN
@@
 	3475 3600 3475 5375
 $Comp
-L Device:R_Small_US R?
+L Device:R_Small_US R3
 U 1 1 5DD2EB95
 P 3750 3500
-F 0 "R?" H 3725 3400 50  0000 R CNN
+F 0 "R3" H 3725 3400 50  0000 R CNN
 F 1 "1k" H 3725 3600 50  0000 R CNN
 F 2 "" H 3750 3500 50  0001 C CNN
@@
 	3750 3600 3750 4925
 $Comp
-L Device:R_Small_US R?
+L Device:R_Small_US R4
 U 1 1 5DD2EDDB
 P 4025 3500
-F 0 "R?" H 4000 3400 50  0000 R CNN
+F 0 "R4" H 4000 3400 50  0000 R CNN
 F 1 "1k" H 4000 3600 50  0000 R CNN
 F 2 "" H 4025 3500 50  0001 C CNN
@@
 Wire Wire Line
 	1600 3200 1600 4250
+$Comp
+L Connector_Generic:Conn_01x02 J8
+U 1 1 5DD0F56F
+P 6650 1500
+F 0 "J8" H 6730 1492 50  0000 L CNN
+F 1 "Power" H 6730 1401 50  0000 L CNN
+F 2 "" H 6650 1500 50  0001 C CNN
+F 3 "~" H 6650 1500 50  0001 C CNN
+	1    6650 1500
+	1    0    0    -1
+$EndComp
 $EndSCHEMATC

Commit message: Detail components (BOM, schematics)
Parts:
- added BT1: Battery_Cell, symbol Device:Battery_Cell
- added PCB1: CHARGER, symbol board:CHARGER
- added PCB2: BOOSTER, symbol board:BOOSTER
- J7: value Power -> Power connection
- J8: value Power -> Power switch
Connections:
- net +5V: now also PCB2.4 (+5V)
- net GND: now also J7.1 (Pin_1), PCB1.2 (SUPPLY-), PCB2.3 (GND)
- net at J8.1 (Pin_1): now also BT1.1 (+), PCB1.4 (BAT+)
- net at J8.2 (Pin_2): now also PCB2.1 (BAT+)
- net at J7.2 (Pin_2): now also PCB1.1 (SUPPLY+)
- new net: BT1.2 (-), PCB1.3 (BAT-), PCB2.2 (BAT-)
Other:
- note added: "Note: block the VCC FTDI\nPTH with a drop of glue"
- moved on the sheet: B1, J1, J2, J3, J4, J5, J6, J7, J8, R1, R10, R2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
